File: bm1370.kicad_sch (KiCad schematic)
At the start: 78 parts, among them J2 Conn_01x06, U19 BM1370_mode1, U20 BM1370_mode1, U25 BM1370_mode1, U26 BM1370_mode1, U35 TXU0304PW, U8 25MHz

Commit message: updated power stage placements
Parts:
- removed C11, C13, C15, C17: 100µ/10V, Capacitor_SMD:C_1210_3225Metric, symbol Device:C
- removed C25, C49, C53, C55, C59, C82, C83: 100n, Capacitor_SMD:C_0805_2012Metric, symbol Device:C
- removed C26, C27, C29, C31: 10µ/25V, Capacitor_SMD:C_0805_2012Metric, symbol Device:C
- removed C28, C30, C32, C33, C34, C35, C36, C37, C38, C40, C41, C42, C43, C44, C46, C47, C50, C51, C52, C54, C56, C57, C58, C60, C62, C63, C64, C66, C67, C68, C69, C70, C71, C72, C73, C74, C75, C76, C77, C78, C79, C80, C93, C94: 1µ/25V, Capacitor_SMD:C_0805_2012Metric, symbol Device:C
- removed J2: Conn_01x06, Connector_PinHeader_1.27mm:PinHeader_1x06_P1.27mm_Vertical, symbol Connector_Generic:Conn_01x06
- removed R19, R20, R21, R22, R23: 10k, Resistor_SMD:R_0805_2012Metric, symbol Device:R
- removed R44, R45, R46, R47: 1k, Resistor_SMD:R_0805_2012Metric, symbol Device:R
- removed R49, R50, R51: 2k, Resistor_SMD:R_0805_2012Metric, symbol Device:R
- removed U19, U20, U25, U26: BM1370_mode1, qaxe:BM1370_JB, symbol mylib7:BM1368_mode1
- removed U35: TXU0304PW, Package_SO:TSSOP-14_4.4x5mm_P0.65mm, symbol mylib7:TXU0304
- removed U8: 25MHz, Oscillator:Oscillator_SMD_EuroQuartz_XO32-4Pin_3.2x2.5mm, symbol Oscillator:ASDMB-xxxMHz
Connections:
- no-connect marks 25 -> 0
Other:
- title: BRAIINS AXE -> (none)
