File: CONTROL.kicad_sch (KiCad schematic)
At the start: 68 parts, among them J1 RJ45_Hanrun_HR911105A_Horizon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, J9 Conn_01x10, M1 Fan_4pin, M2 Fan_4pin, U12 W5500, U17 TMP1075, U30 T-Display-S3, U32 EMC2302-1, U33 TXU0102-DCU, U37 TMP1075, U38 TMP1075, X1 TXM25M0004322JBDDO00T

Commit message: rp2350 connections
Parts:
- removed C229: 100n/0.7mm, Capacitor_SMD:C_0805_2012Metric, symbol Device:C
- removed U17, U37: TMP1075, myfootprints:TMP1075-DRL, symbol mylib7:TMP1075-DRL-SOT563
- removed U38: TMP1075, Nerd8:TMP1075-DRL, symbol mylib7:TMP1075-DRL-SOT563
- added C148: 2.2uF, Capacitor_SMD:C_0603_1608Metric, symbol Parts:root_0_CAP_NOPOL_Parts.DbLib
- added C184: 10µ, Capacitor_SMD:C_0805_2012Metric, symbol Device:C
- added R154, R155: 33R, Resistor_SMD:R_0603_1608Metric, symbol Parts:root_0_Resistor_Parts.DbLib
- added R61: 10k, Resistor_SMD:R_0603_1608Metric, symbol Device:R
- added R62, R63: 0R, Resistor_SMD:R_0603_1608Metric, symbol Device:R
- added R64: 10R, Resistor_SMD:R_0603_1608Metric, symbol Device:R
- added R65, R66: 2.7k, Resistor_SMD:R_0603_1608Metric, symbol Device:R
- added SW1: SW_Omron_B3F-315x, Button_Switch_THT:SW_SPST_Omron_B3F-315x_Angled, symbol Switch:SW_Omron_B3FS
- added U1, U13: TMP102xxDRL, Package_TO_SOT_SMD:SOT-563, symbol Sensor_Temperature:TMP102xxDRL
- C87, C88: footprint Capacitor_SMD:C_0805_2012Metric -> Capacitor_SMD:C_0603_1608Metric
- J9: value Conn_01x10 -> DISP
- R36, R43, R44: footprint Resistor_SMD:R_0805_2012Metric -> Resistor_SMD:R_0603_1608Metric
Connections:
- net +3V3: now also R61.1, R64.2, R65.1, R66.1, U1.5 (V+), U13.4 (ADD0), U13.5 (V+)
- net 3V3: now also A1.36 (3V3), J9.9 (Pin_9), C184.1
- net GND: now also A1.13 (GND), A1.18 (GND), A1.23 (GND), A1.28 (GND), A1.3 (GND), A1.33 (AGND), A1.38 (GND), A1.8 (GND), J9.10 (Pin_10), C148.2, C184.2, SW1.1, U1.2 (GND), U1.4 (ADD0), U13.2 (GND)
- net LDO_EN: now also R63.1; no longer U30.8 (GPIO13)
- net PWR_EN: now also R62.1; no longer U30.5 (GPIO10)
- net RESET: now also A1.4 (GPIO2); no longer U30.2 (GPIO1)
- net RXD: now also A1.7 (GPIO5); no longer U30.20 (GPIO18)
- net SCL: now also A1.27 (GPIO21), U1.1 (SCL), U13.1 (SCL); no longer U30.22 (GPIO43)
- net SDA: now also A1.26 (GPIO20), U1.6 (SDA), U13.6 (SDA); no longer U30.21 (GPIO44)
- net TXD: now also A1.6 (GPIO4); no longer U30.19 (GPIO17)
- net VR_RDY: no longer U30.6 (GPIO11)
- net W5500_CSN: now also A1.22 (GPIO17)
- net W5500_INT_N: now also A1.29 (GPIO22)
- net W5500_MISO: now also A1.21 (GPIO16)
- net W5500_MOSI: now also R154.2
- net W5500_RST_N: now also A1.31 (GPIO26_ADC0)
- net W5500_SCLK: now also R155.2
- net DISP_SDA: now reaches J9.1 (Pin_1)
- net DISP_SDA: now also A1.9 (GPIO6), R65.2
- net DISP_SCL: now reaches J9.2 (Pin_2)
- net DISP_SCL: now also A1.10 (GPIO7), R66.2
- net at A1.1 (GPIO0): now also R62.2
- net at A1.2 (GPIO1): now also R63.2
- net at A1.24 (GPIO18): now also R155.1
- net at A1.25 (GPIO19): now also R154.1
- net RUN: now reaches A1.30 (RUN)
- net RUN: now also R61.2, SW1.2
- net at A1.35 (ADC_VREF): now also C148.1, R64.1
- no-connect marks 11 -> 8
Other:
- moved on the sheet: A1, C128, C129, C130, C131, C132, C133, C134, C135, C136, C137, C138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

Commit message: fans
Parts:
- removed C102, C103, C96: 100n/0.7mm, Capacitor_SMD:C_0603_1608Metric, symbol Device:C
- removed U32: EMC2302-1, Package_SO:MSOP-10_3x3mm_P0.5mm, symbol mylib7:EMC2302
- removed U33: TXU0102-DCU, Package_SO:VSSOP-8_2.3x2mm_P0.5mm, symbol mylib7:TXU0102DCK
- added C149, C150: 68nF/50V, Capacitor_SMD:C_0603_1608Metric, symbol Device:C
- added D3, D4, D5: STPS1H100A, Diode_SMD:D_SMA, symbol Device:D_Schottky
- added Q1, Q2: BSS138, Package_TO_SOT_SMD:SOT-23, symbol Transistor_FET:BSS138
- added R67, R73, R76, R77, R79: 0R, Resistor_SMD:R_0603_1608Metric, symbol Device:R
- added R68, R71: 100R, Resistor_SMD:R_0603_1608Metric, symbol Device:R
- added R72, R78: NC, Resistor_SMD:R_0603_1608Metric, symbol Device:R
- added R74, R75: 10k, Resistor_SMD:R_0603_1608Metric, symbol Device:R
Connections:
- net +12V: now also D5.1 (K)
- net GND: now also C149.2, C150.2, D3.2 (A), D4.2 (A), D5.2 (A), Q1.2 (S), Q2.2 (S), R74.2, R75.2
- net VR_RDY: now also R67.1
- net at M2.4 (PWM): now also R72.2, R73.2
- net RP_PWM1: now reaches A1.11 (GPIO8)
- net RP_PWM1: now also R78.1, R79.1
- net RP_PWM2: now reaches A1.12 (GPIO9)
- net RP_PWM2: now also R72.1, R77.1
- net RP_TACHO1: now reaches A1.32 (GPIO27_ADC1)
- net RP_TACHO1: now also C149.1, R71.1
- net RP_TACHO2: now reaches A1.34 (GPIO28_ADC2)
- net RP_TACHO2: now also C150.1, R68.1
- net at A1.5 (GPIO3): now also R67.2
- net at M1.4 (PWM): now also R76.2, R78.2
- net TACHO1: no longer names the net of M1.3 (Tacho), R33.2
- net TACHO1: now also D4.1 (K), R71.2
- net TACHO2: no longer names the net of M2.3 (Tacho), R35.2
- net TACHO2: now also D3.1 (K), R68.2
- new net: Q2.1 (G), R75.1, R79.2
- new net: Q1.1 (G), R74.1, R77.2
- new net: Q2.3 (D), R76.1
- new net: Q1.3 (D), R73.1
- no-connect marks 8 -> 6
Other:
- moved on the sheet: M1, M2, R33, R35

Commit message: sch_ should be ready
Parts:
- removed U30: T-Display-S3, myfootprints:T-Display-S3, symbol bitaxe:T-Display-S3
- added R156, R157: 33R, Resistor_SMD:R_0603_1608Metric, symbol Parts:root_0_Resistor_Parts.DbLib
Connections:
- net DISP_ALRT: now reaches J9.3 (Pin_3)
- net DISP_ALRT: now also A1.20 (GPIO15)
- net DISP_CSN: now reaches J9.4 (Pin_4)
- net DISP_CSN: now also A1.17 (GPIO13)
- net DISP_DC: now reaches J9.5 (Pin_5)
- net DISP_DC: now also A1.16 (GPIO12)
- net DISP_RST: now reaches J9.6 (Pin_6)
- net DISP_RST: now also A1.19 (GPIO14)
- net DISP_MOSI: now reaches J9.7 (Pin_7)
- net DISP_MOSI: now also R157.1
- net DISP_SCK: now reaches J9.8 (Pin_8)
- net DISP_SCK: now also R156.1
- net at A1.14 (GPIO10): now also R156.2
- net at A1.15 (GPIO11): now also R157.2
- no-connect marks 6 -> 1
Other:
- moved on the sheet: C144, C145, C146, C147, C149, C150, C185, C189, C87, C88, D3, D4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
