File: CONTROL.kicad_sch (KiCad schematic)
At the start: 93 parts, among them J1 RJ45_Hanrun_HR911105A_Horizon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, J9 DISP, M1 Fan_4pin, M2 Fan_4pin, Q1 BSS138, Q2 BSS138, SW1 SW_Omron_B3F-315x, U1 TMP102xxDRL, U12 W5500, U13 TMP102xxDRL, X1 TXM25M0004322JBDDO00T

Commit message: A RGB connector added
Parts:
- added C153: 22uF/16V, Capacitor_SMD:C_1206_3216Metric, symbol Device:C
- added J5: Conn_01x04_Pin, Connector_PinHeader_2.54mm:PinHeader_1x04_P2.54mm_Vertical, symbol Connector:Conn_01x04_Pin
Connections:
- net +5V: now also C153.1, J5.1 (Pin_1)
- net DISP_SDA: now also J5.2 (Pin_2)
- net GND: now also C153.2, J5.4 (Pin_4)
- no-connect marks 1 -> 2
Other:
- note added: "ARGB 5V connector"
- note added: "DISPLAY CONNECTOR"
- moved on the sheet: J9
