File: power.kicad_sch (KiCad schematic)
At the start: 120 parts, among them J3 Conn_01x01, J4 Conn_01x01, U14 AP3211, U16 CSD95472Q5MC, U3 TPS53647, U36 MCP1824T-1202E, U4 CSD95472Q5MC, U5 CSD95472Q5MC, U6 AP3211, U7 MCP1824T-0802E

Commit message: Change micro symbol to uF
Parts:
- C100, C102: value 10µ/25V -> 10uF/25V
- C105, C108, C113, C118, C182, C6, C8: value 1µ/25V -> 1uF/25V
- C106, C152: value 22µ/16V -> 22uF/16V
- C111, C191, C192, C193, C20, C23, C45, C81, C89: value 22µ/25V -> 22uF/25V
- C119, C120, C183: value 10µ -> 10uF
- C12, C13, C177: value 2.2µ -> 2.2uF
- C186, C187, C188, C48, C84, C86, C90, C91, C95, C97, C98, C99: value 330µ/4V -> 330uF/4V
- C190, C92: value 220µ/25V -> 220uF/25V
- C206, C207, C21, C22, C24, C39: value 100µ/6.3V -> 100uF/6.3V
- C7: value 4.7µ -> 4.7uF
- L3, L6: value 4.7µH/2.3A/2.7A -> 4.7uH/2.3A/2.7A
Changed lines of the file:
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@@
 			)
 		)
-		(property "Value" "22µ/25V"
+		(property "Value" "22uF/25V"
 			(at 320.04 67.31 90)
 			(show_name no)
@@
 			)
 		)
-		(property "Value" "330µ/4V"
+		(property "Value" "330uF/4V"
 			(at 324.866 156.972 90)
 			(show_name no)
@@
 			)
 		)
-		(property "Value" "330µ/4V"
+		(property "Value" "330uF/4V"
 			(at 299.72 157.226 90)
 			(show_name no)
@@
 			)
 		)
-		(property "Value" "330µ/4V"
+		(property "Value" "330uF/4V"
 			(at 335.28 156.972 90)
 			(show_name no)
@@
 			)
 		)
-		(property "Value" "1µ/25V"
+		(property "Value" "1uF/25V"
 			(at 175.895 268.605 0)
 			(show_name no)
@@
 			)
 		)
-		(property "Value" "22µ/25V"
+		(property "Value" "22uF/25V"
 			(at 336.55 67.31 90)
 			(show_name no)
@@
 			)
 		)
-		(property "Value" "100µ/6.3V"
+		(property "Value" "100uF/6.3V"
 			(at 245.11 158.242 90)
 			(show_name no)
@@
 			)
 		)
-		(property "Value" "100µ/6.3V"
+		(property "Value" "100uF/6.3V"
 			(at 259.08 158.242 90)
 			(show_name no)
@@
 			)
 		)
-		(property "Value" "330µ/4V"
+		(property "Value" "330uF/4V"
 			(at 284.48 156.972 90)
 			(show_name no)
@@
 			)
 		)
-		(property "Value" "100µ/6.3V"
+		(property "Value" "100uF/6.3V"
 			(at 251.46 158.242 90)
 			(show_name no)
@@
 			)
 		)
-		(property "Value" "2.2µ"
+		(property "Value" "2.2uF"
 			(at 182.88 95.2499 0)
 			(show_name no)
@@
 			)
 		)
-		(property "Value" "220µ/25V"
+		(property "Value" "220uF/25V"
 			(at 351.155 37.465 90)
 			(show_name no)
@@
 			)
 		)
-		(property "Value" "330µ/4V"
+		(property "Value" "330uF/4V"
 			(at 289.56 156.972 90)
 			(show_name no)
@@
 			)
 		)
-		(property "Value" "2.2µ"
+		(property "Value" "2.2uF"
 			(at 184.15 146.0499 0)
 			(show_name no)
@@
 			)
 		)
-		(property "Value" "22µ/25V"
+		(property "Value" "22uF/25V"
 			(at 303.53 67.31 90)
 			(show_name no)
@@
 			)
 		)
-		(property "Value" "22µ/16V"
+		(property "Value" "22uF/16V"
 			(at 84.201 217.043 0)
 			(show_name no)
@@
 			)
 		)
-		(property "Value" "330µ/4V"
+		(property "Value" "330uF/4V"
 			(at 330.2 156.972 90)
 			(show_name no)
@@
 			)
 		)
-		(property "Value" "22µ/25V"
+		(property "Value" "22uF/25V"
 			(at 353.06 67.31 90)
 			(show_name no)
@@
 			)
 		)
-		(property "Value" "220µ/25V"
+		(property "Value" "220uF/25V"
 			(at 342.265 37.465 90)
 			(show_name no)
@@
 			)
 		)
-		(property "Value" "4.7µH/2.3A/2.7A"
+		(property "Value" "4.7uH/2.3A/2.7A"
 			(at 63.5 256.54 90)
 			(show_name no)
@@
 			)
 		)
-		(property "Value" "330µ/4V"
+		(property "Value" "330uF/4V"
 			(at 314.96 156.718 90)
 			(show_name no)
@@
 			)
 		)
-		(property "Value" "1µ/25V"
+		(property "Value" "1uF/25V"
 			(at 77.47 162.56 90)
 			(show_name no)
@@
 			)
 		)
-		(property "Value" "22µ/25V"
+		(property "Value" "22uF/25V"
 			(at 294.64 67.31 90)
 			(show_name no)
@@
 			)
 		)
-		(property "Value" "2.2µ"
+		(property "Value" "2.2uF"
 			(at 184.15 189.2299 0)
 			(show_name no)
@@
 			)
 		)
-		(property "Value" "10µ/25V"
+		(property "Value" "10uF/25V"
 			(at 27.051 214.503 0)
 			(show_name no)
@@
 			)
 		)
-		(property "Value" "330µ/4V"
+		(property "Value" "330uF/4V"
 			(at 304.8 156.21 90)
 			(show_name no)
@@
 			)
 		)
-		(property "Value" "1µ/25V"
+		(property "Value" "1uF/25V"
 			(at 199.39 36.83 90)
 			(show_name no)
@@
 			)
 		)
-		(property "Value" "10µ"
+		(property "Value" "10uF"
 			(at 264.16 36.83 0)
 			(show_name no)
@@
 			)
 		)
-		(property "Value" "4.7µH/2.3A/2.7A"
+		(property "Value" "4.7uH/2.3A/2.7A"
 			(at 62.23 207.01 90)
 			(show_name no)
@@
 			)
 		)
-		(property "Value" "330µ/4V"
+		(property "Value" "330uF/4V"
 			(at 341.63 156.464 90)
 			(show_name no)
@@
 			)
 		)
-		(property "Value" "4.7µ"
+		(property "Value" "4.7uF"
 			(at 82.55 157.48 90)
 			(show_name no)
@@
 			)
 		)
-		(property "Value" "100µ/6.3V"
+		(property "Value" "100uF/6.3V"
 			(at 278.13 158.496 90)
 			(show_name no)
@@
 			)
 		)
-		(property "Value" "10µ"
+		(property "Value" "10uF"
 			(at 256.54 36.83 0)
 			(show_name no)
@@
 			)
 		)
-		(property "Value" "1µ/25V"
+		(property "Value" "1uF/25V"
 			(at 234.95 268.605 0)
 			(show_name no)
@@
 			)
 		)
-		(property "Value" "22µ/25V"
+		(property "Value" "22uF/25V"
 			(at 312.42 67.31 90)
 			(show_name no)
@@
 			)
 		)
-		(property "Value" "22µ/25V"
+		(property "Value" "22uF/25V"
 			(at 328.93 67.31 90)
 			(show_name no)
@@
 			)
 		)
-		(property "Value" "22µ/16V"
+		(property "Value" "22uF/16V"
 			(at 85.471 266.573 0)
 			(show_name no)
@@
 			)
 		)
-		(property "Value" "10µ/25V"
+		(property "Value" "10uF/25V"
 			(at 28.321 264.033 0)
 			(show_name no)
@@
 			)
 		)
-		(property "Value" "22µ/25V"
+		(property "Value" "22uF/25V"
 			(at 285.75 67.31 90)
 			(show_name no)
@@
 			)
 		)
-		(property "Value" "22µ/25V"
+		(property "Value" "22uF/25V"
 			(at 344.17 67.31 90)
 			(show_name no)
@@
 			)
 		)
-		(property "Value" "330µ/4V"
+		(property "Value" "330uF/4V"
 			(at 309.88 156.972 90)
 			(show_name no)
@@
 			)
 		)
-		(property "Value" "1µ/25V"
+		(property "Value" "1uF/25V"
 			(at 218.44 36.83 90)
 			(show_name no)
@@
 			)
 		)
-		(property "Value" "10µ"
+		(property "Value" "10uF"
 			(at 271.78 36.83 0)
 			(show_name no)
@@
 			)
 		)
-		(property "Value" "330µ/4V"
+		(property "Value" "330uF/4V"
 			(at 320.04 156.464 90)
 			(show_name no)
@@
 			)
 		)
-		(property "Value" "100µ/6.3V"
+		(property "Value" "100uF/6.3V"
 			(at 271.78 158.496 90)
 			(show_name no)
@@
 			)
 		)
-		(property "Value" "1µ/25V"
+		(property "Value" "1uF/25V"
 			(at 238.76 36.83 90)
 			(show_name no)
@@
 			)
 		)
-		(property "Value" "100µ/6.3V"
+		(property "Value" "100uF/6.3V"
 			(at 265.43 158.242 90)
 			(show_name no)
@@
 			)
 		)
-		(property "Value" "330µ/4V"
+		(property "Value" "330uF/4V"
 			(at 294.64 156.464 90)
 			(show_name no)
@@
 			)
 		)
-		(property "Value" "1µ/25V"
+		(property "Value" "1uF/25V"
 			(at 87.63 160.02 90)
 			(show_name no)
