File: power.kicad_sch (KiCad schematic)
At the start: 120 parts, among them J3 Conn_01x01, J4 Conn_01x01, U14 AP3211, U16 CSD95472Q5MC, U3 TPS53647, U36 MCP1824T-1202E, U4 CSD95472Q5MC, U5 CSD95472Q5MC, U6 AP3211, U7 MCP1824T-0802E

Commit message: Add LCSC number to components
Parts:
- C1: LCSC (none) -> C107082
- C100, C102, C119, C120, C183: LCSC (none) -> C318691
- C104, C151: LCSC (none) -> C83170
- C105, C108: LCSC (none) -> C91186
- C106, C152: LCSC (none) -> C105212
- C111, C191, C192, C193, C20, C23, C45, C81, C89: LCSC (none) -> C140122
- C112, C117, C181: LCSC (none) -> C1613
- C113, C118, C182, C6, C8: LCSC (none) -> C59302
- C114, C115, C116: LCSC (none) -> C1653
- C12, C13, C177: LCSC (none) -> C106853
- C14, C16, C178: LCSC (none) -> C694249
- C179, C18, C19, C2, C4, C9: LCSC (none) -> C36911373
- C186, C187, C188, C48, C84, C86, C90, C91, C95, C97, C98, C99: LCSC (none) -> C4982610
- C190, C92: LCSC (none) -> C311610
- C206, C207, C21, C22, C24, C39: LCSC (none) -> C49066
- C3: LCSC (none) -> C107034
- C5: LCSC (none) -> C107070
- C7: LCSC (none) -> C69335
- D2, D6: LCSC (none) -> C96234
- L3, L6: LCSC (none) -> C354606
- R1: LCSC (none) -> C4182677
- R12, R13: LCSC (none) -> C543414
- R2: LCSC (none) -> C276290
- R25, R26, R27, R28, R47, R48: LCSC (none) -> C543407
- R29, R30: LCSC (none) -> C96345
- R3: LCSC (none) -> C105579
- R31: LCSC (none) -> C84376
- R32: LCSC (none) -> C861034
- R34, R70: LCSC (none) -> C728583
- R37, R38: LCSC (none) -> C126901
- R39, R40: LCSC (none) -> C2889384
- R4: LCSC (none) -> C14675
- R5: LCSC (none) -> C25809
- R6: LCSC (none) -> C131052
- R69: LCSC (none) -> C114624
- U14, U6: LCSC (none) -> C154863
- U16, U4, U5: LCSC (none) -> C553137
- U3: LCSC (none) -> C2659348
- U36: LCSC (none) -> C625461
- U7: LCSC (none) -> C625460

Commit message: Add missing LCSC number
Parts:
- R7: LCSC (none) -> C54531329
Changed lines of the file:
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@@
+			)
+		)
+		(property "LCSC" "C54531329"
+			(at 71.12 154.94 90)
+			(hide yes)
+			(show_name no)
+			(do_not_autoplace no)
+			(effects
+				(font
+					(size 1.27 1.27)
+				)
 			)
 		)

Commit message: Use only stock component and unified LCSC capacitor code
Parts:
- C10, C11, C176: LCSC (none) -> C314282
- C101, C107: LCSC (none) -> C49678
- C105, C108: LCSC C91186 -> C5137482
- C106, C152: LCSC C105212 -> C385907
- C109, C110, C180: LCSC (none) -> C36911373
- C111, C191, C192, C193, C20, C23, C45, C81, C89: LCSC C140122 -> C7419439
- C14, C16, C178: LCSC C694249 -> C314282
- C186, C187, C188, C48, C84, C86, C90, C91, C95, C97, C98, C99: LCSC C4982610 -> C528969
- C2, C4, C9: LCSC C36911373 -> C1588
- L1, L2, L4: LCSC (none) -> C20613221
- R1: LCSC C4182677 -> C273769
- R3: LCSC C105579 -> C2907042
- R31: LCSC C84376 -> C2907219
- R32: LCSC C861034 -> C2998081
- R4: LCSC C14675 -> C2907044
Changed lines of the file:
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@@
 			)
 		)
-		(property "LCSC" "C140122"
+		(property "LCSC" "C7419439"
 			(at 316.23 63.5 0)
 			(hide yes)
@@
 			)
 		)
-		(property "LCSC" "C4982610"
+		(property "LCSC" "C528969"
 			(at 325.12 138.43 0)
 			(hide yes)
@@
 			)
 		)
-		(property "LCSC" "C4982610"
+		(property "LCSC" "C528969"
 			(at 299.72 138.43 0)
 			(hide yes)
@@
 			)
 		)
-		(property "LCSC" "C36911373"
+		(property "LCSC" "C1588"
 			(at 48.26 91.44 90)
 			(hide yes)
@@
 			)
 		)
-		(property "LCSC" "C4982610"
+		(property "LCSC" "C528969"
 			(at 335.28 138.43 0)
 			(hide yes)
@@
 			)
 		)
-		(property "LCSC" "C91186"
+		(property "LCSC" "C5137482"
 			(at 174.625 264.795 0)
 			(hide yes)
@@
 			)
 		)
-		(property "LCSC" "C140122"
+		(property "LCSC" "C7419439"
 			(at 332.74 63.5 0)
 			(hide yes)
@@
 			)
 		)
+		(property "LCSC" "C20613221"
+			(at 224.79 80.01 90)
+			(hide yes)
+			(show_name no)
+			(do_not_autoplace no)
+			(effects
+				(font
+					(size 1.27 1.27)
+				)
+			)
+		)
 		(pin "1"
 		)
@@
 			)
 		)
-		(property "LCSC" "C4982610"
+		(property "LCSC" "C528969"
 			(at 284.48 138.43 0)
 			(hide yes)
@@
 			)
 		)
+		(property "LCSC" "C314282"
+			(at 173.99 144.78 0)
+			(hide yes)
+			(show_name no)
+			(do_not_autoplace no)
+			(effects
+				(font
+					(size 1.27 1.27)
+				)
+			)
+		)
 		(pin "2"
 		)
@@
 			)
 		)
-		(property "LCSC" "C694249"
+		(property "LCSC" "C314282"
 			(at 212.09 163.83 90)
 			(hide yes)
@@
 			)
 		)
-		(property "LCSC" "C4982610"
+		(property "LCSC" "C528969"
 			(at 289.56 138.43 0)
 			(hide yes)
@@
 			)
 		)
-		(property "LCSC" "C140122"
+		(property "LCSC" "C7419439"
 			(at 299.72 63.5 0)
 			(hide yes)
@@
 			)
 		)
-		(property "LCSC" "C14675"
+		(property "LCSC" "C2907044"
 			(at 38.1 91.44 0)
 			(hide yes)
@@
 			)
 		)
-		(property "LCSC" "C105212"
+		(property "LCSC" "C385907"
 			(at 81.28 215.9 0)
 			(hide yes)
@@
 			)
 		)
-		(property "LCSC" "C4982610"
+		(property "LCSC" "C528969"
 			(at 330.2 138.43 0)
 			(hide yes)
@@
 			)
 		)
+		(property "LCSC" "C314282"
+			(at 172.72 93.98 0)
+			(hide yes)
+			(show_name no)
+			(do_not_autoplace no)
+			(effects
+				(font
+					(size 1.27 1.27)
+				)
+			)
+		)
 		(pin "2"
 		)
@@
 			)
 		)
+		(property "LCSC" "C314282"
+			(at 173.99 187.96 0)
+			(hide yes)
+			(show_name no)
+			(do_not_autoplace no)
+			(effects
+				(font
+					(size 1.27 1.27)
+				)
+			)
+		)
 		(pin "2"
 		)
@@
 			)
 		)
-		(property "LCSC" "C140122"
+		(property "LCSC" "C7419439"
 			(at 349.25 63.5 0)
 			(hide yes)
@@
 			)
 		)
-		(property "LCSC" "C694249"
+		(property "LCSC" "C314282"
 			(at 212.09 121.92 90)
 			(hide yes)
@@
 			)
 		)
-		(property "LCSC" "C4182677"
+		(property "LCSC" "C273769"
 			(at 118.11 95.885 0)
 			(hide yes)
@@
 			)
 		)
-		(property "LCSC" "C4982610"
+		(property "LCSC" "C528969"
 			(at 314.96 138.43 0)
 			(hide yes)
@@
 			)
 		)
-		(property "LCSC" "C36911373"
+		(property "LCSC" "C1588"
 			(at 129.54 133.35 90)
 			(hide yes)
@@
 			)
 		)
-		(property "LCSC" "C140122"
+		(property "LCSC" "C7419439"
 			(at 290.83 63.5 0)
 			(hide yes)
@@
 			)
 		)
+		(property "LCSC" "C36911373"
+			(at 234.95 137.16 90)
+			(hide yes)
+			(show_name no)
+			(do_not_autoplace no)
+			(effects
+				(font
+					(size 1.27 1.27)
+				)
+			)
+		)
 		(pin "1"
 		)
@@
 			)
 		)
-		(property "LCSC" "C4982610"
+		(property "LCSC" "C528969"
 			(at 304.8 138.43 0)
 			(hide yes)
@@
 			)
 		)
+		(property "LCSC" "C36911373"
+			(at 233.68 91.44 90)
+			(hide yes)
+			(show_name no)
+			(do_not_autoplace no)
+			(effects
+				(font
+					(size 1.27 1.27)
+				)
+			)
+		)
 		(pin "1"
 		)
@@
 			)
 		)
-		(property "LCSC" "C4982610"
+		(property "LCSC" "C528969"
 			(at 341.63 138.43 0)
 			(hide yes)
@@
 			)
 		)
-		(property "LCSC" "C36911373"
+		(property "LCSC" "C1588"
 			(at 60.96 160.02 90)
 			(hide yes)
@@
 			)
 		)
+		(property "LCSC" "C20613221"
+			(at 226.06 173.99 90)
+			(hide yes)
+			(show_name no)
+			(do_not_autoplace no)
+			(effects
+				(font
+					(size 1.27 1.27)
+				)
+			)
+		)
 		(pin "1"
 		)
@@
 			)
 		)
+		(property "LCSC" "C49678"
+			(at 196.215 263.525 0)
+			(hide yes)
+			(show_name no)
+			(do_not_autoplace no)
+			(effects
+				(font
+					(size 1.27 1.27)
+				)
+			)
+		)
 		(pin "1"
 		)
@@
 			)
 		)
-		(property "LCSC" "C84376"
+		(property "LCSC" "C2907219"
 			(at 130.81 262.89 0)
 			(hide yes)
@@
 			)
 		)
+		(property "LCSC" "C36911373"
+			(at 234.95 185.42 90)
+			(hide yes)
+			(show_name no)
+			(do_not_autoplace no)
+			(effects
+				(font
+					(size 1.27 1.27)
+				)
+			)
+		)
 		(pin "1"
 		)
@@
 			)
 		)
+		(property "LCSC" "C49678"
+			(at 139.065 263.525 0)
+			(hide yes)
+			(show_name no)
+			(do_not_autoplace no)
+			(effects
+				(font
+					(size 1.27 1.27)
+				)
+			)
+		)
 		(pin "1"
 		)
@@
 			)
 		)
-		(property "LCSC" "C91186"
+		(property "LCSC" "C5137482"
 			(at 233.045 264.795 0)
 			(hide yes)
@@
 			)
 		)
-		(property "LCSC" "C140122"
+		(property "LCSC" "C7419439"
 			(at 308.61 63.5 0)
 			(hide yes)
@@
 			)
 		)
-		(property "LCSC" "C140122"
+		(property "LCSC" "C7419439"
 			(at 325.12 63.5 0)
 			(hide yes)
@@
 			)
 		)
-		(property "LCSC" "C105212"
+		(property "LCSC" "C385907"
 			(at 82.55 265.43 0)
 			(hide yes)
@@
 			)
 		)
-		(property "LCSC" "C140122"
+		(property "LCSC" "C7419439"
 			(at 281.94 63.5 0)
 			(hide yes)
@@
 			)
 		)
-		(property "LCSC" "C140122"
+		(property "LCSC" "C7419439"
 			(at 340.36 63.5 0)
 			(hide yes)
@@
 			)
 		)
-		(property "LCSC" "C694249"
+		(property "LCSC" "C314282"
 			(at 210.82 69.85 90)
 			(hide yes)
@@
 			)
 		)
-		(property "LCSC" "C4982610"
+		(property "LCSC" "C528969"
 			(at 309.88 138.43 0)
 			(hide yes)
@@
 			)
 		)
+		(property "LCSC" "C20613221"
+			(at 226.06 130.81 90)
+			(hide yes)
+			(show_name no)
+			(do_not_autoplace no)
+			(effects
+				(font
+					(size 1.27 1.27)
+				)
+			)
+		)
 		(pin "1"
 		)
@@
 			)
 		)
-		(property "LCSC" "C105579"
+		(property "LCSC" "C2907042"
 			(at 31.75 118.11 0)
 			(hide yes)
@@
 			)
 		)
-		(property "LCSC" "C861034"
+		(property "LCSC" "C2998081"
 			(at 68.58 210.82 0)
 			(hide yes)
@@
 			)
 		)
-		(property "LCSC" "C4982610"
+		(property "LCSC" "C528969"
 			(at 320.04 138.43 0)
 			(hide yes)
@@
 			)
 		)
-		(property "LCSC" "C4982610"
+		(property "LCSC" "C528969"
 			(at 294.64 138.43 0)
 			(hide yes)
