File: power.kicad_sch (KiCad schematic)
At the start: 120 parts, among them J3 Conn_01x01, J4 Conn_01x01, U14 AP3211, U16 CSD95472Q5MC, U3 TPS53647, U36 MCP1824T-1202E, U4 CSD95472Q5MC, U5 CSD95472Q5MC, U6 AP3211, U7 MCP1824T-0802E

Commit message: 5V header connectot added
Parts:
- added C153: 22uF/16V, Capacitor_SMD:C_1206_3216Metric, symbol Device:C
- added J5: Conn_01x02_Pin, Connector_PinHeader_2.54mm:PinHeader_1x02_P2.54mm_Vertical, symbol Connector:Conn_01x02_Pin
Connections:
- net +5V: now also C153.1, J5.1 (Pin_1)
- net GND: now also C153.2, J5.2 (Pin_2)

Commit message: A RGB connector added
Parts:
- removed C153: 22uF/16V, Capacitor_SMD:C_1206_3216Metric, symbol Device:C
- removed J5: Conn_01x02_Pin, Connector_PinHeader_2.54mm:PinHeader_1x02_P2.54mm_Vertical, symbol Connector:Conn_01x02_Pin
