File: Asic0.kicad_sch (KiCad schematic)
At the start: 19 parts, among them U2 BM1370_mode1

Commit message: Change micro symbol to uF
Parts:
- C15, C17, C26, C27, C28, C30, C32, C33, C35, C36, C37, C38, C40: value 1µ/25V -> 1uF/25V
- C29: value 10µ/25V -> 10uF/25V
- C31: value 100µ/6.3V -> 100uF/6.3V
Changed lines of the file:
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@@
 			)
 		)
-		(property "Value" "1µ/25V"
+		(property "Value" "1uF/25V"
 			(at 87.63 115.824 90)
 			(show_name no)
@@
 			)
 		)
-		(property "Value" "100µ/6.3V"
+		(property "Value" "100uF/6.3V"
 			(at 140.716 156.972 90)
 			(show_name no)
@@
 			)
 		)
-		(property "Value" "1µ/25V"
+		(property "Value" "1uF/25V"
 			(at 161.544 43.561 90)
 			(show_name no)
@@
 			)
 		)
-		(property "Value" "1µ/25V"
+		(property "Value" "1uF/25V"
 			(at 174.244 43.561 90)
 			(show_name no)
@@
 			)
 		)
-		(property "Value" "10µ/25V"
+		(property "Value" "10uF/25V"
 			(at 122.174 132.842 90)
 			(show_name no)
@@
 			)
 		)
-		(property "Value" "1µ/25V"
+		(property "Value" "1uF/25V"
 			(at 185.674 43.561 90)
 			(show_name no)
@@
 			)
 		)
-		(property "Value" "1µ/25V"
+		(property "Value" "1uF/25V"
 			(at 72.898 108.712 90)
 			(show_name no)
@@
 			)
 		)
-		(property "Value" "1µ/25V"
+		(property "Value" "1uF/25V"
 			(at 134.112 131.572 90)
 			(show_name no)
@@
 			)
 		)
-		(property "Value" "1µ/25V"
+		(property "Value" "1uF/25V"
 			(at 183.134 101.346 90)
 			(show_name no)
@@
 			)
 		)
-		(property "Value" "1µ/25V"
+		(property "Value" "1uF/25V"
 			(at 99.314 43.561 90)
 			(show_name no)
@@
 			)
 		)
-		(property "Value" "1µ/25V"
+		(property "Value" "1uF/25V"
 			(at 87.884 43.561 90)
 			(show_name no)
@@
 			)
 		)
-		(property "Value" "1µ/25V"
+		(property "Value" "1uF/25V"
 			(at 147.574 43.561 90)
 			(show_name no)
@@
 			)
 		)
-		(property "Value" "1µ/25V"
+		(property "Value" "1uF/25V"
 			(at 110.744 43.561 90)
 			(show_name no)
@@
 			)
 		)
-		(property "Value" "1µ/25V"
+		(property "Value" "1uF/25V"
 			(at 197.358 108.712 90)
 			(show_name no)
@@
 			)
 		)
-		(property "Value" "1µ/25V"
+		(property "Value" "1uF/25V"
 			(at 123.444 43.561 90)
 			(show_name no)

Commit message: Add LCSC number to components
Parts:
- C15, C17, C26, C27, C28, C30, C32, C33, C35, C36, C37, C38, C40: LCSC (none) -> C91186
- C29: LCSC (none) -> C318691
- C31: LCSC (none) -> C49066
- R10: LCSC (none) -> C84376
- R9: LCSC (none) -> C95781

Commit message: Use only stock component and unified LCSC capacitor code
Parts:
- C15, C17, C26, C27, C28, C30, C32, C33, C35, C36, C37, C38, C40: LCSC C91186 -> C5137482
- C34: LCSC (none) -> C49678
- R10: LCSC C84376 -> C2907219
Changed lines of the file:
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@@
 			)
 		)
-		(property "LCSC" "C91186"
+		(property "LCSC" "C5137482"
 			(at 91.948 112.014 0)
 			(hide yes)
@@
 			)
 		)
-		(property "LCSC" "C91186"
+		(property "LCSC" "C5137482"
 			(at 162.814 42.926 0)
 			(hide yes)
@@
 			)
 		)
-		(property "LCSC" "C91186"
+		(property "LCSC" "C5137482"
 			(at 175.514 42.926 0)
 			(hide yes)
@@
 			)
 		)
-		(property "LCSC" "C84376"
+		(property "LCSC" "C2907219"
 			(at 174.244 78.486 0)
 			(hide yes)
@@
 			)
 		)
-		(property "LCSC" "C91186"
+		(property "LCSC" "C5137482"
 			(at 186.944 42.926 0)
 			(hide yes)
@@
 			)
 		)
-		(property "LCSC" "C91186"
+		(property "LCSC" "C5137482"
 			(at 78.74 112.522 0)
 			(hide yes)
@@
 			)
 		)
-		(property "LCSC" "C91186"
+		(property "LCSC" "C5137482"
 			(at 137.414 125.984 0)
 			(hide yes)
@@
 			)
 		)
-		(property "LCSC" "C91186"
+		(property "LCSC" "C5137482"
 			(at 187.452 105.156 0)
 			(hide yes)
@@
 			)
 		)
-		(property "LCSC" "C91186"
+		(property "LCSC" "C5137482"
 			(at 100.584 42.926 0)
 			(hide yes)
@@
 			)
 		)
-		(property "LCSC" "C91186"
+		(property "LCSC" "C5137482"
 			(at 89.154 42.926 0)
 			(hide yes)
@@
 			)
 		)
+		(property "LCSC" "C49678"
+			(at 151.003 124.333 0)
+			(hide yes)
+			(show_name no)
+			(do_not_autoplace no)
+			(effects
+				(font
+					(size 1.27 1.27)
+				)
+			)
+		)
 		(pin "1"
 		)
@@
 			)
 		)
-		(property "LCSC" "C91186"
+		(property "LCSC" "C5137482"
 			(at 148.844 42.926 0)
 			(hide yes)
@@
 			)
 		)
-		(property "LCSC" "C91186"
+		(property "LCSC" "C5137482"
 			(at 112.014 42.926 0)
 			(hide yes)
@@
 			)
 		)
-		(property "LCSC" "C91186"
+		(property "LCSC" "C5137482"
 			(at 200.152 104.902 0)
 			(hide yes)
@@
 			)
 		)
-		(property "LCSC" "C91186"
+		(property "LCSC" "C5137482"
 			(at 128.524 42.926 0)
 			(hide yes)
